File: main.kicad_sch (KiCad schematic)
At the start: 21 parts, among them J1 Conn_01x03_Socket, J2 Conn_01x02_Socket, U1 MP1584EN-LF-Z, U2 LED_Voltmeter_2D

Commit message: docs: add blank line in readme for spacing
Parts:
- C1: value 10u -> C_Small
- C2: value 100n -> C_Small
- C3: value 22pF -> C_Small
- C4: value 150pF -> C_Small
- C5: value 10n -> C_Small
- D1: value ~ -> D_Zener_Small
- L1: value 15u -> L_Small
- R1, R3, R4: value 100k -> R_US
- R2, R7, R8: value 24.9K -> R_US
- R5: value 210k -> R_US
- R6: value 40.2k -> R_US
Other:
- moved on the sheet: C3, D1
